File: Macropad/PCB/Macropad.kicad_pcb (KiCad board)
At the start: 2 copper layers, 85.1 x 46.7 mm, 9 parts, among them SW1 SW_Push, SW2 SW_Push, SW3 SW_Push, SW4 SW_Push, SW5 SW_Push, SW6 RotaryEncoder_Switch, U1 XIAO-RP2040-DIP

Commit message: Cleaned up the files and organised them into folders (CAD, PCD, Firmware).
Connections:
- SW6 pad B: GND -> Net-(U1-GPIO29/ADC3/A3)
- SW6 pad S2: +5V -> GND
- U1 pad 4: unconnected-(U1-GPIO29/ADC3/A3-Pad4) -> Net-(U1-GPIO29/ADC3/A3)
Routing:
- net Net-(U1-GPIO29/ADC3/A3): track 0.00 -> 68.9 mm, vias 0 -> 2
- net +5V: track 74.8 -> 30.5 mm
- net GND: track 123.8 -> 151.3 mm
Changed lines of the file:
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@@
 	(net 11 "unconnected-(U1-3V3-Pad12)")
 	(net 12 "Net-(U1-GPIO7{slash}SCL)")
-	(net 13 "unconnected-(U1-GPIO29{slash}ADC3{slash}A3-Pad4)")
+	(net 13 "Net-(U1-GPIO29{slash}ADC3{slash}A3)")
 	(net 14 "Net-(U1-GPIO6{slash}SDA)")
 	(net 15 "unconnected-(U1-GPIO27{slash}ADC1{slash}A1-Pad2)")
@@
 			(layers "*.Cu" "*.Mask")
 			(remove_unused_layers no)
-			(net 2 "GND")
+			(net 13 "Net-(U1-GPIO29{slash}ADC3{slash}A3)")
 			(pinfunction "B")
 			(pintype "passive")
@@
 			(layers "*.Cu" "*.Mask")
 			(remove_unused_layers no)
-			(net 4 "+5V")
+			(net 2 "GND")
 			(pinfunction "S2")
 			(pintype "passive")
@@
 			(layers "F.Cu" "F.Mask")
 			(roundrect_rratio 0.1)
-			(net 13 "unconnected-(U1-GPIO29{slash}ADC3{slash}A3-Pad4)")
+			(net 13 "Net-(U1-GPIO29{slash}ADC3{slash}A3)")
 			(pinfunction "GPIO29/ADC3/A3")
 			(pintype "passive")
@@
 			(layers "*.Cu" "*.Mask")
 			(remove_unused_layers no)
-			(net 13 "unconnected-(U1-GPIO29{slash}ADC3{slash}A3-Pad4)")
+			(net 13 "Net-(U1-GPIO29{slash}ADC3{slash}A3)")
 			(pinfunction "GPIO29/ADC3/A3")
 			(pintype "passive")
@@
 	)
 	(segment
-		(start 164.465 49.86)
-		(end 164.465 52.07)
+		(start 164.465 33.02)
+		(end 169.545 38.1)
 		(width 0.2)
 		(layer "B.Cu")
@@
 	)
 	(segment
-		(start 173.725 38.1)
-		(end 173.725 40.6)
+		(start 126.365 52.07)
+		(end 145.415 52.07)
 		(width 0.2)
 		(layer "B.Cu")
@@
 	)
 	(segment
-		(start 173.725 40.6)
-		(end 164.465 49.86)
+		(start 140.2 28)
+		(end 139.9425 28.2575)
 		(width 0.2)
 		(layer "B.Cu")
@@
 	)
 	(segment
-		(start 164.465 33.02)
-		(end 169.545 38.1)
+		(start 175.94145 35.88355)
+		(end 187.94145 35.88355)
 		(width 0.2)
 		(layer "B.Cu")
@@
 	)
 	(segment
-		(start 126.365 52.07)
-		(end 145.415 52.07)
+		(start 139.9425 28.2575)
+		(end 131.445 28.2575)
 		(width 0.2)
 		(layer "B.Cu")
@@
 	)
 	(segment
-		(start 140.2 28)
-		(end 139.9425 28.2575)
+		(start 186.525 37.3)
+		(end 187.94145 35.88355)
 		(width 0.2)
 		(layer "B.Cu")
@@
 	)
 	(segment
-		(start 139.9425 28.2575)
-		(end 131.445 28.2575)
+		(start 164.465 52.07)
+		(end 179.235 37.3)
+		(width 0.2)
+		(layer "B.Cu")
+		(net 2)
+	)
+	(segment
+		(start 173.725 38.1)
+		(end 175.94145 35.88355)
+		(width 0.2)
+		(layer "B.Cu")
+		(net 2)
+	)
+	(segment
+		(start 179.235 37.3)
+		(end 186.525 37.3)
 		(width 0.2)
 		(layer "B.Cu")
@@
 	)
 	(segment
-		(start 188.225 35.6)
-		(end 178.81875 26.19375)
-		(width 0.2)
-		(layer "B.Cu")
-		(net 4)
-	)
-	(segment
 		(start 147.6 33.96875)
 		(end 147.79375 33.775)
@@
 	)
 	(segment
-		(start 178.81875 26.19375)
-		(end 147.79375 26.19375)
-		(width 0.2)
-		(layer "B.Cu")
-		(net 4)
-	)
-	(segment
 		(start 147.79375 26.19375)
 		(end 147.3175 25.7175)
@@
 	)
 	(segment
+		(start 147.1 43.1)
+		(end 143.8 43.1)
+		(width 0.2)
+		(layer "F.Cu")
+		(net 13)
+	)
+	(via
+		(at 147.1 43.1)
+		(size 0.6)
+		(drill 0.3)
+		(layers "F.Cu" "B.Cu")
+		(net 13)
+	)
+	(via
+		(at 143.8 43.1)
+		(size 0.6)
+		(drill 0.3)
+		(layers "F.Cu" "B.Cu")
+		(net 13)
+	)
+	(segment
+		(start 147.1 43.1)
+		(end 147 43.1)
+		(width 0.2)
+		(layer "B.Cu")
+		(net 13)
+	)
+	(segment
+		(start 143.701 43.001)
+		(end 143.8 43.1)
+		(width 0.2)
+		(layer "B.Cu")
+		(net 13)
+	)
+	(segment
+		(start 171.225 43.1)
+		(end 147.1 43.1)
+		(width 0.2)
+		(layer "B.Cu")
+		(net 13)
+	)
+	(segment
+		(start 116.74519 43.001)
+		(end 143.701 43.001)
+		(width 0.2)
+		(layer "B.Cu")
+		(net 13)
+	)
+	(segment
+		(start 115.142 34.4005)
+		(end 116.205 33.3375)
+		(width 0.2)
+		(layer "B.Cu")
+		(net 13)
+	)
+	(segment
+		(start 115.142 41.39781)
+		(end 115.142 34.4005)
+		(width 0.2)
+		(layer "B.Cu")
+		(net 13)
+	)
+	(segment
+		(start 116.74519 43.001)
+		(end 115.142 41.39781)
+		(width 0.2)
+		(layer "B.Cu")
+		(net 13)
+	)
+	(segment
+		(start 173.725 40.6)
+		(end 171.225 43.1)
+		(width 0.2)
+		(layer "B.Cu")
+		(net 13)
+	)
+	(segment
